Commit message: feat(inspire_description): prefix parameter for multi-gripper URDFs
Add optional `prefix:=''` param to the `gripper` xacro macro so that
multiple gripper instances can coexist in one URDF without duplicate
link/joint name errors. Default empty string preserves full backwards
compatibility; standalone URDF still emits unprefixed names.

File: src/inspire_description/urdf/inspire_gripper.urdf.xacro (robot description, xacro)
@@ -2,5 +2,5 @@
 <robot xmlns:xacro="http://www.ros.org/wiki/xacro" name="gripper_robot">
     <!-- 定义宏 -->
-    <xacro:macro name="gripper" params="parent_link">
+    <xacro:macro name="gripper" params="parent_link prefix:=''">
         <!-- gripper关节上下限 (0 = open as-modeled, positive closes) -->
         <xacro:property name="joint_lower_bound" value="0" />
@@ -9,5 +9,5 @@
         <xacro:property name="joint_velocity" value="1.0" />
         <!-- gripper -->
-        <link name="gripper_base_link">
+        <link name="${prefix}gripper_base_link">
             <inertial>
                 <origin xyz="-2.6792E-06 1.4343E-05 -0.040955" rpy="0 0 0" />
@@ -31,10 +31,10 @@
             </collision>
         </link>
-        <joint name="gripper_base_joint" type="fixed">
+        <joint name="${prefix}gripper_base_joint" type="fixed">
             <origin xyz="0 0 0.008" rpy="0 0 0" />
             <parent link="${parent_link}" />
-            <child link="gripper_base_link" />
+            <child link="${prefix}gripper_base_link" />
         </joint>
-        <link name="gripper_Link1">
+        <link name="${prefix}gripper_Link1">
             <inertial>
                 <origin xyz="0.0001 0.0085832 0.013664" rpy="0 0 0" />
@@ -60,13 +60,13 @@
         <!-- Driven joint for the 4-bar parallel gripper mechanism.
              Positive rotation about +X closes the jaws (Link1 rotates toward vertical). -->
-        <joint name="gripper_joint1" type="revolute">
+        <joint name="${prefix}gripper_joint1" type="revolute">
             <origin xyz="0 -0.04 0.09" rpy="0.8663 0 0" />
-            <parent link="gripper_base_link" />
-            <child link="gripper_Link1" />
+            <parent link="${prefix}gripper_base_link" />
+            <child link="${prefix}gripper_Link1" />
             <axis xyz="-1 0 0" />
             <limit lower="${joint_lower_bound}" upper="${joint_upper_bound}"
                    effort="${joint_effort}" velocity="${joint_velocity}" />
         </joint>
-        <link name="gripper_Link2">
+        <link name="${prefix}gripper_Link2">
             <inertial>
                 <origin xyz="9.9997E-05 0.011846 0.011367" rpy="0 0 0" />
@@ -91,14 +91,14 @@
         </link>
         <!-- Follower joint: mirrors joint1 to keep Link2 (fingertip) parallel to the base. -->
-        <joint name="gripper_joint2" type="revolute">
+        <joint name="${prefix}gripper_joint2" type="revolute">
             <origin xyz="0 0.022341 0.035565" rpy="-0.8663 0 0" />
-            <parent link="gripper_Link1" />
-            <child link="gripper_Link2" />
+            <parent link="${prefix}gripper_Link1" />
+            <child link="${prefix}gripper_Link2" />
             <axis xyz="-1 0 0" />
             <limit lower="${-joint_upper_bound}" upper="${-joint_lower_bound}"
                    effort="${joint_effort}" velocity="${joint_velocity}" />
-            <mimic joint="gripper_joint1" multiplier="-1.0" offset="0.0" />
+            <mimic joint="${prefix}gripper_joint1" multiplier="-1.0" offset="0.0" />
         </joint>
-        <link name="gripper_Link3">
+        <link name="${prefix}gripper_Link3">
             <inertial>
                 <origin xyz="0.0001 -0.0085832 0.013664" rpy="0 0 0" />
@@ -123,14 +123,14 @@
         </link>
         <!-- Mirrored driven joint: closes together with joint1 on the opposite side. -->
-        <joint name="gripper_joint3" type="revolute">
+        <joint name="${prefix}gripper_joint3" type="revolute">
             <origin xyz="0 0.04 0.09" rpy="-0.8663 0 0" />
-            <parent link="gripper_base_link" />
-            <child link="gripper_Link3" />
+            <parent link="${prefix}gripper_base_link" />
+            <child link="${prefix}gripper_Link3" />
             <axis xyz="-1 0 0" />
             <limit lower="${-joint_upper_bound}" upper="${-joint_lower_bound}"
                    effort="${joint_effort}" velocity="${joint_velocity}" />
-            <mimic joint="gripper_joint1" multiplier="-1.0" offset="0.0" />
+            <mimic joint="${prefix}gripper_joint1" multiplier="-1.0" offset="0.0" />
         </joint>
-        <link name="gripper_Link4">
+        <link name="${prefix}gripper_Link4">
             <inertial>
                 <origin xyz="9.9999E-05 -0.011846 0.011367" rpy="0 0 0" />
@@ -155,19 +155,19 @@
         </link>
         <!-- Follower joint: mirrors joint3 to keep Link4 (fingertip) parallel to the base. -->
-        <joint name="gripper_joint4" type="revolute">
+        <joint name="${prefix}gripper_joint4" type="revolute">
             <origin xyz="0 -0.022341 0.035565" rpy="0.8663 0 0" />
-            <parent link="gripper_Link3" />
-            <child link="gripper_Link4" />
+            <parent link="${prefix}gripper_Link3" />
+            <child link="${prefix}gripper_Link4" />
             <axis xyz="-1 0 0" />
             <limit lower="${joint_lower_bound}" upper="${joint_upper_bound}"
                    effort="${joint_effort}" velocity="${joint_velocity}" />
-            <mimic joint="gripper_joint1" multiplier="1.0" offset="0.0" />
+            <mimic joint="${prefix}gripper_joint1" multiplier="1.0" offset="0.0" />
         </joint>
         <!-- gripper tip virtual link (TCP), 0.1522 m along +Z from the gripper base. -->
-        <link name="gripper_tip_link"/>
-        <joint name="gripper_tip_joint" type="fixed">
+        <link name="${prefix}gripper_tip_link"/>
+        <joint name="${prefix}gripper_tip_joint" type="fixed">
             <origin xyz="0 0 0.1522" rpy="0 0 0" />
-            <parent link="gripper_base_link" />
-            <child link="gripper_tip_link" />
+            <parent link="${prefix}gripper_base_link" />
+            <child link="${prefix}gripper_tip_link" />
         </joint>
     </xacro:macro>
